File: PCB/coolboard.kicad_pcb (KiCad board)
At the start: 2 copper layers, 21 x 51 mm, 38 parts, among them J1 USB_C_Receptacle_USB2.0_14P, J2 Conn_01x20, J3 Conn_01x20, J4 Conn_01x03, SW1 SW_Push, U1 RP2040, U2 MCP1700x-330xxTT, U4 W25Q16JVUXIQ TR, Y1 12 MHz

Commit message: Update production zip file with latest changes
Parts:
- added R9: 100, Capacitor_SMD:C_0402_1005Metric, F.Cu at (139.0, 110.7)
- added U3: IRM-H6xxT, OptoDevice:Everlight_IRM-H6xxT, F.Cu at (134.2, 112.5)
- G***: moved to B.Cu
- moved G*** 4.25 mm to (130.4, 109.5), turned to 90 degrees
- moved R8 3.99 mm to (140.8, 110.8)
- moved D1 2.69 mm to (140.3, 113.9)
Connections:
- J2 pad 20: GPIO15 -> GND
Routing:
- net +3V3: track 90.0 -> 94.8 mm
- net GND: track 46.8 -> 50.3 mm
- net GPIO16: track 9.05 -> 12.0 mm
- net GPIO15: track 21.8 -> 20.0 mm
- net Net-(D1-DIN): track 3.54 -> 1.74 mm
- net Net-(U3-Vcc): track 0.00 -> 1.63 mm
